Commit message: feat: hardware updates with no differential drive

File: src/gungnir_description/urdf/gungnir.ros2_control.xacro (robot description, xacro)
@@ -36,9 +36,8 @@
         <state_interface name="velocity"/>
       </joint>
-      <!--
       <joint name="joint_4">
         <command_interface name="velocity">
-          <param name="min">-3.2</param>
-          <param name="max">3.2</param>
+          <param name="min">-2</param>
+          <param name="max">2</param>
         </command_interface>
         <state_interface name="position">
@@ -47,4 +46,5 @@
         <state_interface name="velocity"/>
       </joint>
+  <!--
       <joint name="joint_5">
         <command_interface name="velocity">

File: src/gungnir_description/urdf/gungnir.urdf.xacro (robot description, xacro)
@@ -4,4 +4,5 @@
   <!-- helper macro -->
   <xacro:include filename="$(find gungnir_description)/urdf/inc/create_link.xacro"/>
+  <xacro:include filename="$(find gungnir_description)/urdf/inc/create_link_no_mesh.xacro"/>
   <xacro:create_link
       link_name="base_link"
@@ -32,10 +33,10 @@
       mesh_name="link_3"
   />
-<!--
-  <xacro:create_link
+  <xacro:create_link_no_mesh
       link_name="link_4"
-      xyz_offset="0 0 0.077"
+      xyz_offset="0 0 -.2"
       rpy_offset="0 0 0"
   />
+<!--
   <xacro:create_link
       link_name="link_5"
@@ -84,12 +85,12 @@
     <limit effort="1000.0" lower="${-pi}" upper="${pi}" velocity="2.5"/>
   </joint>
-  <!--
   <joint name="joint_4" type="revolute">
     <parent link="link_3"/>
     <child link="link_4"/>
-    <origin xyz="0.519 0 0" rpy="0 ${pi} ${pi}"/>
+    <origin xyz="0 0 0" rpy="0 ${pi/2} 0"/>
     <axis xyz="0 0 1"/>
     <limit effort="1000.0" lower="${-pi}" upper="${pi}" velocity="2.5"/>
   </joint>
+  <!--
   <joint name="joint_5" type="revolute">
     <parent link="link_4"/>

Commit message: feat: added differential joint

File: src/gungnir_description/urdf/gungnir.ros2_control.xacro (robot description, xacro)
@@ -46,9 +46,8 @@
         <state_interface name="velocity"/>
       </joint>
-  <!--
       <joint name="joint_5">
         <command_interface name="velocity">
-          <param name="min">-3.2</param>
-          <param name="max">3.2</param>
+          <param name="min">-3.14</param>
+          <param name="max">3.14</param>
         </command_interface>
         <state_interface name="position">
@@ -59,6 +58,6 @@
       <joint name="joint_6">
         <command_interface name="velocity">
-          <param name="min">-3.2</param>
-          <param name="max">3.2</param>
+          <param name="min">-3.1</param>
+          <param name="max">3.14</param>
         </command_interface>
         <state_interface name="position">
@@ -66,5 +65,5 @@
         </state_interface>
         <state_interface name="velocity"/>
-      </joint> -->
+      </joint>
     </ros2_control>
   </xacro:macro>

File: src/gungnir_description/urdf/gungnir.urdf.xacro (robot description, xacro)
@@ -35,19 +35,19 @@
   <xacro:create_link_no_mesh
       link_name="link_4"
-      xyz_offset="0 0 -.2"
+      xyz_offset="0 0 0"
+      rpy_offset="0 0 0"
+  />
+  <xacro:create_link_no_mesh
+      link_name="link_5"
+      xyz_offset="0 0 0"
+      rpy_offset="0 0 0"
+  />
+  <xacro:create_link_no_mesh
+      link_name="link_6"
+      xyz_offset="0 0 0."
       rpy_offset="0 0 0"
   />
 <!--
-  <xacro:create_link
-      link_name="link_5"
-      xyz_offset="0 0 0.113"
-      rpy_offset="0 0 0"
-  />
-  <xacro:create_link
-      link_name="link_6"
-      xyz_offset="0 0 0.086"
-      rpy_offset="0 0 0"
-  /> -->
-  <!-- <link name="ft_frame"
+ <link name="ft_frame"
     xyz_offset="0 0 0"
     rpy_offset="0 0 0"
@@ -92,9 +92,8 @@
     <limit effort="1000.0" lower="${-pi}" upper="${pi}" velocity="2.5"/>
   </joint>
-  <!--
   <joint name="joint_5" type="revolute">
     <parent link="link_4"/>
     <child link="link_5"/>
-    <origin xyz="0.0 0 0.188" rpy="${pi/2} ${pi} ${pi/2}"/>
+    <origin xyz="0 0 ${upperarm_length}" rpy="0 ${pi/2} 0"/>
     <axis xyz="0 0 1"/>
     <limit effort="1000.0" lower="${-pi}" upper="${pi}" velocity="2.5"/>
@@ -103,8 +102,9 @@
     <parent link="link_5"/>
     <child link="link_6"/>
-    <origin xyz="0.0 0 0.246" rpy="0 ${-pi/2} 0"/>
+    <origin xyz="0.0 0 0" rpy="0 ${-pi/2} 0"/>
     <axis xyz="0 0 1"/>
     <limit effort="1000.0" lower="${-pi}" upper="${pi}" velocity="2.5"/>
   </joint>
+  <!--
   <joint name="joint-ft_frame" type="fixed">
     <parent link="link_6"/>

File: src/gungnir_description/urdf/robot.urdf.xacro (robot description, xacro)
@@ -5,5 +5,5 @@
   <xacro:include filename="$(find gungnir_description)/urdf/gungnir.ros2_control.xacro"/>
   <xacro:property name="upperarm_length" value="0.415"/>
-  <xacro:property name="forearm_length" value="0"/>
+  <xacro:property name="forearm_length" value="0.300"/>
   <!-- create link fixed to the "world" -->
   <link name="world"/>
